Commit message: Added CUDA support, observation and action formatting w/ added parameters

File: urdf/test.ros2_control.xacro (robot description, xacro)
@@ -14,13 +14,8 @@
   </joint>
   <link name="thigh_link" />
-  <joint name="knee" type="revolute">
-    <parent link="thigh_link" />
-    <child link="knee_link" />
-    <limit effort="100.0" velocity="100.0" lower="-3.14159" upper="3.14159" />
-  </joint>
-  <link name="knee_link" />
   <ros2_control name="Test" type="system">
     <hardware>
       <plugin>mock_components/GenericSystem</plugin>
+      <param name="calculate_dynamics">true</param>
     </hardware>
     <joint name="hip">
@@ -40,19 +35,23 @@
       <state_interface name="effort" />
     </joint>
-    <joint name="knee">
-      <command_interface name="position" />
-      <command_interface name="velocity" />
-      <command_interface name="effort" />
-      <state_interface name="position" />
-      <state_interface name="velocity" />
-      <state_interface name="effort" />
-    </joint>
     <sensor name="imu">
-      <state_interface name="angular_velocity.x" />
-      <state_interface name="angular_velocity.y" />
-      <state_interface name="angular_velocity.z" />
-      <state_interface name="linear_acceleration.x" />
-      <state_interface name="linear_acceleration.y" />
-      <state_interface name="linear_acceleration.z" />
+      <state_interface name="angular_velocity.x">
+        <param name="initial_value">0.0</param>
+      </state_interface>
+      <state_interface name="angular_velocity.y">
+        <param name="initial_value">0.0</param>
+      </state_interface>
+      <state_interface name="angular_velocity.z">
+        <param name="initial_value">-9.81</param>
+      </state_interface>
+      <state_interface name="linear_acceleration.x">
+        <param name="initial_value">0.0</param>
+      </state_interface>
+      <state_interface name="linear_acceleration.y">
+        <param name="initial_value">0.0</param>
+      </state_interface>
+      <state_interface name="linear_acceleration.z">
+        <param name="initial_value">0.0</param>
+      </state_interface>
     </sensor>
   </ros2_control>
